File: kicad/releases/20261027-2346-rev-a-ssi/hastadaq/hastadaq.kicad_pcb (KiCad board)
At the start: 2 copper layers, 62 x 89.3 mm, 44 parts, among them J1 IMU via Qwiic breakout (The P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, J10 SBUS IN (RC receiver): GND, V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, J11 SSI2: RM08 encoder (3V3, GND,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, J2 GAUGE BOARD LOOM (J_I2C): GND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, J3 ENC1 SPI port: MT6835 (pitch), J4 ENC2 SPI port: MT6835, J5 ENC3 SPI port: RLS Orbis (or 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, J6 SSI1: RM08 encoder (3V3, GND,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, J7 SBUS servo header 3x6 (6 plug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, J8 Main supply cable (2x4): VSUP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, J9 TRIG_OUT pull-up (1x5), Q1 2N3904 NPN (TO-92, pin 1 E, 2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, U1 Pimoroni Pico Plus 2 (header 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, U2 Pololu D42V55F8 8.4V 5A buck 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, U3 SparkFun BabyBuck 5V (AP63357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, U4 FOD817A opto (TRIG_IN)

Commit message: Main board: owner silkscreen edits, re-export fab files (Gerbers, drills, zip)
Co-Authored-By: Claude Sonnet 5.5 <noreply@anthropic.com>
Other:
- board text added: "WT Model MCU"
